Commit message: urdf & rviz setting study

File: dummy1_description/urdf/base.urdf.xacro (robot description, xacro)
@@ -1,13 +1,19 @@
 <?xml version="1.0"?>
 <robot xmlns:xacro="http://www.ros.org/wiki/xacro">
-    <xacro:property name="base_width" value="0.31"/>
-    <xacro:property name="base_length" value="0.42"/>
-    <xacro:property name="base_height" value="0.18"/>
-    <xacro:property name="wheel_radius" value="0.10"/>
+    <xacro:property name="base_width" value="0.200"/>
+    <xacro:property name="base_length" value="0.445"/>
+    <xacro:property name="base_height" value="0.039"/>
+    <xacro:property name="wheel_radius" value="0.073"/>
     <xacro:property name="wheel_width" value="0.04"/>
     <xacro:property name="wheel_ygap" value="0.025"/>
-    <xacro:property name="wheel_zoff" value="0.05"/>
-    <xacro:property name="wheel_xoff" value="0.12"/>
-    <xacro:property name="caster_xoff" value="0.14"/>
+    <xacro:property name="wheel_zoff" value="0.025"/>
+    <xacro:property name="wheel_xoff" value="0.183"/>
+    <xacro:property name="bar_yoff" value="0.06"/>
+    <material name="Gray">
+        <color rgba="0.5 0.5 0.5 1.0"/>
+    </material>
+    <material name="Green">
+        <color rgba="0.0 1.0 0.0 1.0"/>
+    </material>
         <link name="base_link">
             <visual>
@@ -27,39 +33,129 @@
             <origin xyz="0.0 0.0 ${-(wheel_radius+wheel_zoff)}" rpy="0.0 0.0 0.0"/>
         </joint>
-        <xacro:macro name="wheel" params="prefix x_reflect y_reflect">
-            <link name="${prefix}_link">
-                <visual>
-                    <origin xyz="0.0 0.0 0.0" rpy="${pi/2} 0.0 0.0"/>
-                    <geometry>
-                        <cylinder radius="${wheel_radius}" length="${wheel_width}"/>
-                    </geometry>
-                    <material name="Gray">
-                        <color rgba="0.5 0.5 0.5 1.0"/>
-                    </material>
-                </visual>
-            </link>
-            <joint name="${prefix}_joint" type="continuous">
-                <parent link="base_link"/>
-                <child link="${prefix}_link"/>
-                <axis xyz="0.0 1.0 0.0"/>
-                <origin xyz="${x_reflect*wheel_xoff} ${y_reflect*(base_width/2+wheel_ygap)} ${-wheel_zoff}" rpy="0.0 0.0 0.0"/>
-            </joint>
-        </xacro:macro>
-        <xacro:wheel prefix="drivewhl_l" x_reflect="-1" y_reflect="1"/>
-        <xacro:wheel prefix="drivewhl_r" x_reflect="-1" y_reflect="-1"/>
-        <link name="front_caster">
+        <link name="laser">
             <visual>
                 <geometry>
-                    <sphere radius="${(wheel_radius+wheel_zoff-(base_height/2))}"/>
+                    <cylinder radius="0.04" length="0.04"/>
                 </geometry>
-                <material name="Cyan">
-                    <color rgba="0.0 1 1 1"/>
-                </material>
             </visual>
         </link>
-        <joint name="caster_joint" type="fixed">
-            <origin xyz="${caster_xoff} 0.0 ${-(base_height/2)}" rpy="0.0 0.0 0.0"/>
+        <joint name="laser_joint" type="fixed">
+            <origin xyz="0.065 0.0 0.0960" />
             <parent link="base_link"/>
-            <child link="front_caster"/>
+            <child link="laser"/>
         </joint>
+    <xacro:macro name="wheel" params="prefix x_reflect y_reflect">
+        <link name="${prefix}_link">
+            <visual>
+                <origin xyz="0.0 0.0 0.0" rpy="${pi/2} 0.0 0.0"/>
+                <geometry>
+                    <cylinder radius="${wheel_radius}" length="${wheel_width}"/>
+                </geometry>
+                <material name="Gray"/>
+            </visual>
+        </link>
+        <joint name="${prefix}_joint" type="continuous">
+            <parent link="base_link"/>
+            <child link="${prefix}_link"/>
+            <axis xyz="0.0 1.0 0.0"/>
+            <origin xyz="${x_reflect*wheel_xoff} ${y_reflect*(base_width/2+wheel_ygap)} ${-wheel_zoff}" rpy="0.0 0.0 0.0"/>
+        </joint>
+    </xacro:macro>
+        <!-- <xacro:wheel prefix="driveFwhl_l" x_reflect="1" y_reflect="1"/> -->
+        <!-- <xacro:wheel prefix="driveFwhl_r" x_reflect="1" y_reflect="-1"/> -->
+        <xacro:wheel prefix="driveRwhl_l" x_reflect="-1" y_reflect="1"/>
+        <xacro:wheel prefix="driveRwhl_r" x_reflect="-1" y_reflect="-1"/>
+    <link name="steer_link">
+        <visual>
+            <origin xyz="-0.02 0.0 0.0" />
+            <geometry>
+                <box size="0.03 0.01995 0.005"/>
+            </geometry>
+            <material name="Gray"/>
+        </visual>
+    </link>
+    <joint name="steer_joint" type="revolute">
+        <origin xyz="0.0 0.0 0.0" rpy="0.0 0.0 0.0"/>
+        <parent link="base_link"/>
+        <child link="steer_link"/>
+        <axis xyz="0.0 0.0 1"/>
+        <limit lower="-0.5" upper="0.5" effort="100.0" velocity="10.0"/>
+    </joint>
+    <link name="front_L_bar_link">
+        <visual>
+            <origin xyz="-0.02 0.0 0.0" rpy="0.0 0.0 0.0"/>
+            <geometry>
+                <box size="0.03 0.01995 0.005"/>
+            </geometry>
+            <material name="Green"/>
+        </visual>
+    </link>
+    <link name="front_R_bar_link">
+        <visual>
+            <origin xyz="-0.02 0.0 0.0" rpy="0.0 0.0 0.0"/>
+            <geometry>
+                <box size="0.03 0.01995 0.005"/>
+            </geometry>
+            <material name="Green"/>
+        </visual>
+    </link>
+    <joint name="front_R_bar_joint" type="revolute">
+        <origin xyz="0.0 ${-bar_yoff} 0.0" rpy="0.0 0.0 0.0"/>
+        <parent link="base_link"/>
+        <child link="front_R_bar_link"/>
+        <axis xyz="0.0 0.0 1"/>
+        <limit lower="-0.5" upper="0.5" effort="100" velocity="10.0"/>
+    </joint>
+    <joint name="front_L_bar_joint" type="revolute">
+        <origin xyz="0.0 ${bar_yoff} 0.0" rpy="0.0 0.0 0.0"/>
+        <parent link="base_link"/>
+        <child link="front_L_bar_link"/>
+        <axis xyz="0.0 0.0 1"/>
+        <limit lower="-0.5" upper="0.5" effort="100" velocity="10.0"/>
+    </joint>
+    <link name="front_L_wheel_link">
+        <visual>
+            <origin rpy="${pi/2} 0.0 0.0"/>
+            <geometry>
+                <cylinder radius="${wheel_radius}" length="${wheel_width}"/>
+            </geometry>
+            <material name="Gray"/>
+        </visual>
+    </link>
+    <joint name="front_L_wheel_joint" type="continuous">
+        <parent link="front_L_bar_link"/>
+        <child link="front_L_wheel_link"/>
+        <axis xyz="0.0 1.0 0.0"/>
+        <origin xyz="${wheel_xoff} ${(base_width/2-bar_yoff+(wheel_width/2))} ${-wheel_zoff}" rpy="0.0 0.0 0.0"/>
+    </joint>
+    <link name="front_R_wheel_link">
+        <visual>
+            <origin rpy="${pi/2} 0 0"/>
+            <geometry>
+                <cylinder radius="${wheel_radius}" length="${wheel_width}"/>
+            </geometry>
+            <material name="Gray"/>
+        </visual>
+    </link>
+    <joint name="front_R_wheel_joint" type="continuous">
+        <parent link="front_R_bar_link"/>
+        <child link="front_R_wheel_link"/>
+        <axis xyz="0.0 1.0 0.0"/>
+        <origin xyz="${wheel_xoff} ${-1*((base_width/2)-bar_yoff+(wheel_width/2))} ${-wheel_zoff}" rpy="0.0 0.0 0.0"/>
+    </joint>
+    <link name="ackermann_bar_link">
+        <visual>
+            <geometry>
+                <box size="0.015 0.15 0.01"/>
+            </geometry>
+            <material name="Green"/>
+        </visual>
+    </link>
+    <joint name="ackermann_joint" type="revolute">
+        <limit lower="-0.5" upper="0.5" effort="100" velocity="10"/>
+        <axis xyz="0.0 0.0 1"/>
+        <parent link="steer_link"/>
+        <child link="ackermann_bar_link"/>
+        <origin xyz="-0.04 0.0 0.0"/>
+    </joint>
 </robot>

Commit message: launch file edit

File: dummy1_description/urdf/base.urdf.xacro (robot description, xacro)
@@ -159,3 +159,15 @@
         <origin xyz="-0.04 0.0 0.0"/>
     </joint>
+    <link name="inu_link">
+        <visual>
+            <geometry>
+                <box size="0.1 0.1 0.1"/>
+            </geometry>
+        </visual>
+    </link>
+    <joint name="imu_joint" type="fixed">
+        <parent link="base_link"/>
+        <child link="imu_link"/>
+        <origin xyz="0.0 0.0 0.1"/>
+    </joint>
 </robot>

Commit message: description pkg update

File: dummy1_description/urdf/base.urdf.xacro (robot description, xacro)
@@ -1,4 +1,4 @@
 <?xml version="1.0"?>
-<robot xmlns:xacro="http://www.ros.org/wiki/xacro">
+<robot name="dummy1" xmlns:xacro="http://www.ros.org/wiki/xacro">
     <xacro:property name="base_width" value="0.200"/>
     <xacro:property name="base_length" value="0.445"/>
@@ -159,5 +159,5 @@
         <origin xyz="-0.04 0.0 0.0"/>
     </joint>
-    <link name="inu_link">
+    <link name="imu_link">
         <visual>
             <geometry>

Commit message: odometry setting

File: dummy1_description/urdf/base.urdf.xacro (robot description, xacro)
@@ -16,4 +16,5 @@
         <color rgba="0.0 1.0 0.0 1.0"/>
     </material>
+        <link name="base_footprint"/>
         <link name="base_link">
             <visual>
@@ -27,8 +28,7 @@
             </visual>
         </link>
-        <link name="base_footprint"/>
         <joint name="base_joint" type="fixed">
-            <parent link="base_link"/>
-            <child link="base_footprint"/>
+            <parent link="base_footprint"/>
+            <child link="base_link"/>
             <origin xyz="0.0 0.0 ${-(wheel_radius+wheel_zoff)}" rpy="0.0 0.0 0.0"/>
         </joint>

Commit message: motor change & PID setting & typo fix

File: dummy1_description/urdf/base.urdf.xacro (robot description, xacro)
@@ -165,4 +165,9 @@
             </geometry>
         </visual>
+        <collision>
+            <geometry>
+                <box size="0.1 0.1 0.1"/>
+            </geometry>
+        </collision>
     </link>
     <joint name="imu_joint" type="fixed">

Commit message: urdf fix

File: dummy1_description/urdf/base.urdf.xacro (robot description, xacro)
@@ -1,12 +1,12 @@
 <?xml version="1.0"?>
 <robot name="dummy1" xmlns:xacro="http://www.ros.org/wiki/xacro">
-    <xacro:property name="base_width" value="0.200"/>
-    <xacro:property name="base_length" value="0.445"/>
+    <xacro:property name="base_width" value="0.130"/>
+    <xacro:property name="base_length" value="0.185"/>
     <xacro:property name="base_height" value="0.039"/>
-    <xacro:property name="wheel_radius" value="0.073"/>
-    <xacro:property name="wheel_width" value="0.04"/>
+    <xacro:property name="wheel_radius" value="0.0365"/>
+    <xacro:property name="wheel_width" value="0.035"/>
     <xacro:property name="wheel_ygap" value="0.025"/>
     <xacro:property name="wheel_zoff" value="0.025"/>
-    <xacro:property name="wheel_xoff" value="0.183"/>
+    <xacro:property name="wheel_xoff" value="0.175"/>
     <xacro:property name="bar_yoff" value="0.06"/>
     <material name="Gray">
@@ -31,10 +31,11 @@
             <parent link="base_footprint"/>
             <child link="base_link"/>
-            <origin xyz="0.0 0.0 ${-(wheel_radius+wheel_zoff)}" rpy="0.0 0.0 0.0"/>
+            <origin xyz="0.0 0.0 ${wheel_radius + wheel_zoff}" rpy="0.0 0.0 0.0"/>
         </joint>
         <link name="laser">
             <visual>
+                <!-- <origin xyz="0.0 0.0 0.0" /> -->
                 <geometry>
-                    <cylinder radius="0.04" length="0.04"/>
+                    <cylinder radius="0.0325" length="0.04"/>
                 </geometry>
             </visual>
@@ -59,5 +60,5 @@
             <child link="${prefix}_link"/>
             <axis xyz="0.0 1.0 0.0"/>
-            <origin xyz="${x_reflect*wheel_xoff} ${y_reflect*(base_width/2+wheel_ygap)} ${-wheel_zoff}" rpy="0.0 0.0 0.0"/>
+            <origin xyz="${x_reflect*wheel_xoff/2} ${y_reflect*(base_width/2+wheel_ygap)} ${-wheel_zoff}" rpy="0.0 0.0 0.0"/>
         </joint>
     </xacro:macro>
@@ -127,5 +128,5 @@
         <child link="front_L_wheel_link"/>
         <axis xyz="0.0 1.0 0.0"/>
-        <origin xyz="${wheel_xoff} ${(base_width/2-bar_yoff+(wheel_width/2))} ${-wheel_zoff}" rpy="0.0 0.0 0.0"/>
+        <origin xyz="${wheel_xoff/2} ${(base_width/2-bar_yoff+(wheel_width/2))} ${-wheel_zoff}" rpy="0.0 0.0 0.0"/>
     </joint>
     <link name="front_R_wheel_link">
@@ -142,5 +143,5 @@
         <child link="front_R_wheel_link"/>
         <axis xyz="0.0 1.0 0.0"/>
-        <origin xyz="${wheel_xoff} ${-1*((base_width/2)-bar_yoff+(wheel_width/2))} ${-wheel_zoff}" rpy="0.0 0.0 0.0"/>
+        <origin xyz="${wheel_xoff/2} ${-1*((base_width/2)-bar_yoff+(wheel_width/2))} ${-wheel_zoff}" rpy="0.0 0.0 0.0"/>
     </joint>
     <link name="ackermann_bar_link">
@@ -162,10 +163,10 @@
         <visual>
             <geometry>
-                <box size="0.1 0.1 0.1"/>
+                <box size="0.01 0.01 0.01"/>
             </geometry>
         </visual>
         <collision>
             <geometry>
-                <box size="0.1 0.1 0.1"/>
+                <box size="0.01 0.01 0.01"/>
             </geometry>
         </collision>
@@ -174,5 +175,5 @@
         <parent link="base_link"/>
         <child link="imu_link"/>
-        <origin xyz="0.0 0.0 0.1"/>
+        <origin xyz="0.035 0.0 0.05"/>
     </joint>
 </robot>

Commit message: fix urdf

File: dummy1_description/urdf/base.urdf.xacro (robot description, xacro)
@@ -2,11 +2,11 @@
 <robot name="dummy1" xmlns:xacro="http://www.ros.org/wiki/xacro">
     <xacro:property name="base_width" value="0.130"/>
-    <xacro:property name="base_length" value="0.185"/>
+    <xacro:property name="base_length" value="0.3"/>
     <xacro:property name="base_height" value="0.039"/>
     <xacro:property name="wheel_radius" value="0.0365"/>
     <xacro:property name="wheel_width" value="0.035"/>
-    <xacro:property name="wheel_ygap" value="0.025"/>
+    <xacro:property name="wheel_ygap" value="0.020"/>
     <xacro:property name="wheel_zoff" value="0.025"/>
-    <xacro:property name="wheel_xoff" value="0.175"/>
+    <xacro:property name="wheel_xoff" value="0.183"/>
     <xacro:property name="bar_yoff" value="0.06"/>
     <material name="Gray">
